File: lcd_backpack.sch (EAGLE design)
At the start: 36 parts, among them IC1 LM2936DT-3.0, X1 BU-SMB-V, X2 BU-SMB-V, X3 BU-SMB-V

Commit message: fixed the USB connector to digikey 609-4618-1-nd
Parts:
- removed CN1: (no value), adafruit:USBMINIB
- added J1: SMARTPRJ_MYCON2_USB-MINI-B, Arduino_Leonardo-REV3b_lbr:SMARTPRJ_MYCON2_USB-MINI-B
Connections:
- removed net N$35: TR3.4, X3.2
- removed net N$36: TR2.4, X2.2
- removed net N$37: TR1.4, X1.2
- net GND: now also J1.GND, J1.SH1, J1.SH2, J1.SH3, J1.SH4, J1.SH5, J1.SH6, TR1.4, TR2.4, TR3.4, X1.2, X2.2, X3.2; no longer CN1.GND
- net N$1: now also J1.D+, R10.2; no longer CN1.D+, R9.2
- net N$2: now also J1.D-, R9.2; no longer CN1.D-, R10.2
- net N$3: now also J1.VBUS; no longer CN1.VBUS
Changed lines of the file:
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@@
 <part name="U$1" library="ref-packages" deviceset="SI5351" device=""/>
 <part name="U$2" library="adafruit" deviceset="ATMEGA32U4" device="-AU"/>
-<part name="CN1" library="adafruit" deviceset="USB" device="MINIB"/>
 <part name="C1" library="rcl" deviceset="C-EU" device="C0805" value="1uF"/>
 <part name="C2" library="rcl" deviceset="C-EU" device="C0805" value="22p"/>
@@
 <part name="GND3" library="supply1" deviceset="GND" device=""/>
 <part name="GND4" library="supply1" deviceset="GND" device=""/>
+<part name="GND5" library="supply1" deviceset="GND" device=""/>
 <part name="GND6" library="supply1" deviceset="GND" device=""/>
 <part name="GND7" library="supply1" deviceset="GND" device=""/>
 <part name="GND8" library="supply1" deviceset="GND" device=""/>
 <part name="GND9" library="supply1" deviceset="GND" device=""/>
+<part name="GND10" library="supply1" deviceset="GND" device=""/>
 <part name="GND11" library="supply1" deviceset="GND" device=""/>
 <part name="GND12" library="supply1" deviceset="GND" device=""/>
+<part name="GND13" library="supply1" deviceset="GND" device=""/>
 <part name="GND14" library="supply1" deviceset="GND" device=""/>
 <part name="GND15" library="supply1" deviceset="GND" device=""/>
@@
 <part name="GND28" library="supply1" deviceset="GND" device=""/>
 <part name="+3V13" library="supply1" deviceset="+3V3" device=""/>
+<part name="J1" library="Arduino_Leonardo-REV3b_lbr" deviceset="SMARTPRJ_MYCON2_USB-MINI-B" device=""/>
+<part name="GND29" library="supply1" deviceset="GND" device=""/>
 </parts>
 <sheets>
@@
 <instance part="U$1" gate="G$1" x="144.78" y="7.62"/>
 <instance part="U$2" gate="G$1" x="38.1" y="33.02"/>
-<instance part="CN1" gate="G$1" x="-50.8" y="45.72"/>
 <instance part="C1" gate="G$1" x="7.62" y="40.64" rot="R270"/>
 <instance part="C2" gate="G$1" x="-2.54" y="30.48" rot="R270"/>
@@
 <instance part="GND3" gate="1" x="76.2" y="58.42" rot="R90"/>
 <instance part="GND4" gate="1" x="71.12" y="104.14" rot="R180"/>
+<instance part="GND5" gate="1" x="195.58" y="5.08"/>
 <instance part="GND6" gate="1" x="116.84" y="101.6"/>
 <instance part="GND7" gate="1" x="-2.54" y="76.2" rot="R270"/>
 <instance part="GND8" gate="1" x="-10.16" y="99.06"/>
 <instance part="GND9" gate="1" x="182.88" y="45.72"/>
+<instance part="GND10" gate="1" x="195.58" y="25.4"/>
 <instance part="GND11" gate="1" x="78.74" y="101.6"/>
 <instance part="GND12" gate="1" x="182.88" y="25.4"/>
+<instance part="GND13" gate="1" x="195.58" y="45.72"/>
 <instance part="GND14" gate="1" x="154.94" y="0"/>
 <instance part="GND15" gate="1" x="-40.64" y="99.06"/>
@@
 <instance part="GND28" gate="1" x="165.1" y="40.64"/>
 <instance part="+3V13" gate="G$1" x="165.1" y="53.34"/>
+<instance part="J1" gate="G$1" x="-55.88" y="45.72" rot="MR0"/>
+<instance part="GND29" gate="1" x="-71.12" y="30.48"/>
 </instances>
 <busses>
 </busses>
 <nets>
-<net name="N$3" class="0">
-<segment>
-<pinref part="U$2" gate="G$1" pin="VBUS"/>
-<pinref part="CN1" gate="G$1" pin="VBUS"/>
-<wire x1="15.24" y1="71.12" x2="-40.64" y2="71.12" width="0.1524" layer="91"/>
-<wire x1="-40.64" y1="71.12" x2="-40.64" y2="50.8" width="0.1524" layer="91"/>
-<junction x="15.24" y="71.12"/>
-</segment>
-</net>
 <net name="GND" class="0">
 <segment>
@@
 <pinref part="GND1" gate="1" pin="GND"/>
 <wire x1="2.54" y1="40.64" x2="0" y2="40.64" width="0.1524" layer="91"/>
-</segment>
-<segment>
-<pinref part="CN1" gate="G$1" pin="GND"/>
-<pinref part="GND2" gate="1" pin="GND"/>
-<wire x1="-40.64" y1="40.64" x2="-38.1" y2="40.64" width="0.1524" layer="91"/>
-<wire x1="-38.1" y1="40.64" x2="-38.1" y2="35.56" width="0.1524" layer="91"/>
 </segment>
 <segment>
@@
 </segment>
 <segment>
+<pinref part="TR1" gate="G$1" pin="4"/>
+<pinref part="GND13" gate="1" pin="GND"/>
+<wire x1="195.58" y1="48.26" x2="195.58" y2="50.8" width="0.1524" layer="91"/>
+<pinref part="X1" gate="G1" pin="2"/>
+<wire x1="203.2" y1="53.34" x2="203.2" y2="50.8" width="0.1524" layer="91"/>
+<wire x1="203.2" y1="50.8" x2="195.58" y2="50.8" width="0.1524" layer="91"/>
+<junction x="195.58" y="50.8"/>
+</segment>
+<segment>
+<pinref part="TR2" gate="G$1" pin="4"/>
+<pinref part="GND10" gate="1" pin="GND"/>
+<wire x1="195.58" y1="27.94" x2="195.58" y2="30.48" width="0.1524" layer="91"/>
+<pinref part="X2" gate="G1" pin="2"/>
+<wire x1="195.58" y1="30.48" x2="203.2" y2="30.48" width="0.1524" layer="91"/>
+<wire x1="203.2" y1="30.48" x2="203.2" y2="33.02" width="0.1524" layer="91"/>
+<junction x="195.58" y="30.48"/>
+</segment>
+<segment>
+<pinref part="TR3" gate="G$1" pin="4"/>
+<pinref part="GND5" gate="1" pin="GND"/>
+<wire x1="195.58" y1="7.62" x2="195.58" y2="10.16" width="0.1524" layer="91"/>
+<pinref part="X3" gate="G1" pin="2"/>
+<wire x1="195.58" y1="10.16" x2="203.2" y2="10.16" width="0.1524" layer="91"/>
+<wire x1="203.2" y1="10.16" x2="203.2" y2="12.7" width="0.1524" layer="91"/>
+<junction x="195.58" y="10.16"/>
+</segment>
+<segment>
 <pinref part="X4" gate="-2" pin="1"/>
 <pinref part="GND26" gate="1" pin="GND"/>
@@
 <pinref part="C9" gate="G$1" pin="2"/>
 <pinref part="GND28" gate="1" pin="GND"/>
+</segment>
+<segment>
+<pinref part="GND2" gate="1" pin="GND"/>
+<pinref part="J1" gate="G$1" pin="GND"/>
+<wire x1="-43.18" y1="40.64" x2="-38.1" y2="40.64" width="0.1524" layer="91"/>
+<wire x1="-38.1" y1="40.64" x2="-38.1" y2="35.56" width="0.1524" layer="91"/>
+</segment>
+<segment>
+<pinref part="J1" gate="G$1" pin="SH1"/>
+<wire x1="-68.58" y1="48.26" x2="-71.12" y2="48.26" width="0.1524" layer="91"/>
+<wire x1="-71.12" y1="48.26" x2="-71.12" y2="45.72" width="0.1524" layer="91"/>
+<pinref part="J1" gate="G$1" pin="SH6"/>
+<wire x1="-71.12" y1="45.72" x2="-71.12" y2="43.18" width="0.1524" layer="91"/>
+<wire x1="-71.12" y1="43.18" x2="-71.12" y2="40.64" width="0.1524" layer="91"/>
+<wire x1="-71.12" y1="40.64" x2="-71.12" y2="38.1" width="0.1524" layer="91"/>
+<wire x1="-71.12" y1="38.1" x2="-71.12" y2="35.56" width="0.1524" layer="91"/>
+<wire x1="-71.12" y1="35.56" x2="-68.58" y2="35.56" width="0.1524" layer="91"/>
+<pinref part="J1" gate="G$1" pin="SH5"/>
+<wire x1="-68.58" y1="38.1" x2="-71.12" y2="38.1" width="0.1524" layer="91"/>
+<pinref part="J1" gate="G$1" pin="SH4"/>
+<wire x1="-68.58" y1="40.64" x2="-71.12" y2="40.64" width="0.1524" layer="91"/>
+<pinref part="J1" gate="G$1" pin="SH3"/>
+<wire x1="-68.58" y1="43.18" x2="-71.12" y2="43.18" width="0.1524" layer="91"/>
+<pinref part="J1" gate="G$1" pin="SH2"/>
+<wire x1="-68.58" y1="45.72" x2="-71.12" y2="45.72" width="0.1524" layer="91"/>
+<wire x1="-71.12" y1="35.56" x2="-71.12" y2="33.02" width="0.1524" layer="91"/>
+<pinref part="GND29" gate="1" pin="GND"/>
+<junction x="-71.12" y="35.56"/>
+<junction x="-71.12" y="38.1"/>
+<junction x="-71.12" y="40.64"/>
+<junction x="-71.12" y="43.18"/>
+<junction x="-71.12" y="45.72"/>
 </segment>
 </net>
@@
 </segment>
 </net>
-<net name="N$1" class="0">
-<segment>
-<pinref part="CN1" gate="G$1" pin="D+"/>
-<pinref part="R9" gate="G$1" pin="2"/>
-<wire x1="-40.64" y1="48.26" x2="-10.16" y2="48.26" width="0.1524" layer="91"/>
-</segment>
-</net>
-<net name="N$2" class="0">
-<segment>
-<pinref part="R10" gate="G$1" pin="2"/>
-<pinref part="CN1" gate="G$1" pin="D-"/>
-<wire x1="-20.32" y1="45.72" x2="-40.64" y2="45.72" width="0.1524" layer="91"/>
-</segment>
-</net>
 <net name="N$44" class="0">
 <segment>
@@
 </segment>
 </net>
-<net name="N$35" class="0">
-<segment>
-<pinref part="TR3" gate="G$1" pin="4"/>
-<pinref part="X3" gate="G1" pin="2"/>
-<wire x1="195.58" y1="10.16" x2="203.2" y2="10.16" width="0.1524" layer="91"/>
-<wire x1="203.2" y1="10.16" x2="203.2" y2="12.7" width="0.1524" layer="91"/>
-</segment>
-</net>
-<net name="N$36" class="0">
-<segment>
-<pinref part="TR2" gate="G$1" pin="4"/>
-<pinref part="X2" gate="G1" pin="2"/>
-<wire x1="195.58" y1="30.48" x2="203.2" y2="30.48" width="0.1524" layer="91"/>
-<wire x1="203.2" y1="30.48" x2="203.2" y2="33.02" width="0.1524" layer="91"/>
-</segment>
-</net>
-<net name="N$37" class="0">
-<segment>
-<pinref part="TR1" gate="G$1" pin="4"/>
-<pinref part="X1" gate="G1" pin="2"/>
-<wire x1="203.2" y1="53.34" x2="203.2" y2="50.8" width="0.1524" layer="91"/>
-<wire x1="203.2" y1="50.8" x2="195.58" y2="50.8" width="0.1524" layer="91"/>
-</segment>
-</net>
+<net name="N$3" class="0">
+<segment>
+<pinref part="U$2" gate="G$1" pin="VBUS"/>
+<wire x1="15.24" y1="71.12" x2="-35.56" y2="71.12" width="0.1524" layer="91"/>
+<wire x1="-35.56" y1="71.12" x2="-35.56" y2="50.8" width="0.1524" layer="91"/>
+<pinref part="J1" gate="G$1" pin="VBUS"/>
+<wire x1="-35.56" y1="50.8" x2="-43.18" y2="50.8" width="0.1524" layer="91"/>
+</segment>
+</net>
+<net name="N$1" class="0">
+<segment>
+<pinref part="R10" gate="G$1" pin="2"/>
+<pinref part="J1" gate="G$1" pin="D+"/>
+<wire x1="-20.32" y1="45.72" x2="-43.18" y2="45.72" width="0.1524" layer="91"/>
+</segment>
+</net>
+<net name="N$2" class="0">
+<segment>
+<pinref part="J1" gate="G$1" pin="D-"/>
+<pinref part="R9" gate="G$1" pin="2"/>
+<wire x1="-43.18" y1="48.26" x2="-10.16" y2="48.26" width="0.1524" layer="91"/>
+</segment>
+</net>
